File: hardware/p1/uc.kicad_sch (KiCad schematic)
At the start: 44 parts, among them J1 Conn_01x05_Socket, J2 USB_B, U1 STM32H733VGTx, U2 USBLC6-2P6, Y1 25MHz

Commit message: Started PC app development
Parts:
- added C22: 10n, Capacitor_SMD:C_0603_1608Metric, symbol Device:C
- added TP12: TestPoint, TestPoint:TestPoint_Pad_D1.0mm, symbol Connector:TestPoint
- TP1, TP10, TP11, TP2, TP3, TP4, TP6, TP7, TP8, TP9: footprint (none) -> TestPoint:TestPoint_Pad_D1.0mm
Connections:
- net GND: now also Y1.2 (G), Y1.4 (G), C22.1
- net NRST: now also C22.2
- net VBAT: now also TP12.1
